File: small-stm32/small-stm32.kicad_pcb (KiCad board)
At the start: 4 copper layers, 17.8 x 21 mm, 42 parts, among them J1 USB_C_Receptacle, J3 QWIIC, U2 STM32G0B1CBUxN, Y1 8Mhz SMD2520-4P

Commit message: update-2025-12-08
Parts:
- U3: value ~ -> SGM6029; footprint Package_CSP:WLCSP-6_1.4x1.0mm_P0.4mm -> seeed-stuff:WLCSP-0.74×1.09-6B
- moved G*** 5.85 mm to (87.8, 65.8)
- moved R9 3.40 mm to (90.2, 60.2), turned to 0 degrees
- moved C4 3.03 mm to (93.7, 60.6)
- turned L1 to 0 degrees
- turned U3 to 180 degrees
Connections:
- net Net-(U3-MODE) renamed /MODE
- net Net-(U3-SW) renamed /SW
Routing:
- net +3V3: track 58.0 -> 59.6 mm, vias 10 -> 8
- net VBUS: track 20.1 -> 19.6 mm
